Commit message: fix the most egregious bugs. still needs some more tuning

File: robot_urdf/robot1/robot.urdf (robot description, URDF)
Before this commit: robot robot1, 1 links, 0 joints
Links:
- added link 375__round_id__875__od_radial_bearing__217_3239, mass 0.0136078; collision mesh filename=package://assets/375__round_id__875__od_radial_bearing__217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; visual mesh filename=package://assets/375__round_id__875__od_radial_bearing__217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
- added link 375__round_id__875__od_radial_bearing__217_3239_2, mass 0.0136078; collision mesh filename=package://assets/375__round_id__875__od_radial_bearing__217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; visual mesh filename=package://assets/375__round_id__875__od_radial_bearing__217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
- added link 375__round_id__875__od_radial_bearing__217_3239_3, mass 0.0136078; collision mesh filename=package://assets/375__round_id__875__od_radial_bearing__217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; visual mesh filename=package://assets/375__round_id__875__od_radial_bearing__217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
- added link 375__round_id__875__od_radial_bearing__217_3239_4, mass 0.0136078; collision mesh filename=package://assets/375__round_id__875__od_radial_bearing__217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; visual mesh filename=package://assets/375__round_id__875__od_radial_bearing__217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
- added link 375__round_id__875__od_radial_bearing__217_3239_5, mass 0.0136078; collision mesh filename=package://assets/375__round_id__875__od_radial_bearing__217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; visual mesh filename=package://assets/375__round_id__875__od_radial_bearing__217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
- added link bottom_enclosure, mass 1e-09; collision mesh filename=package://assets/bottom_enclosure.stl; visual mesh filename=package://assets/bottom_enclosure.stl
- added link headtop, mass 1e-09; collision mesh filename=package://assets/headtop.stl; collision mesh filename=package://assets/neckconnector.stl
- added link hex_socket_head_cap_screw_m4x0_70_x_6__52230e09e6b8162f7a31d58ec48e066b, mass 0.00135184; collision mesh filename=package://assets/hex_socket_head_cap_screw_m4x0_70_x_6__522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; visual mesh filename=package://assets/hex_socket_head_cap_screw_m4x0_70_x_6__522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
- added link hex_socket_head_cap_screw_m4x0_70_x_6__52230e09e6b8162f7a31d58ec48e066b_2, mass 0.00135184; collision mesh filename=package://assets/hex_socket_head_cap_screw_m4x0_70_x_6__522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; visual mesh filename=package://assets/hex_socket_head_cap_screw_m4x0_70_x_6__522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
- added link hex_socket_head_cap_screw_m4x0_70_x_6__52230e09e6b8162f7a31d58ec48e066b_3, mass 0.00135184; collision mesh filename=package://assets/hex_socket_head_cap_screw_m4x0_70_x_6__522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; visual mesh filename=package://assets/hex_socket_head_cap_screw_m4x0_70_x_6__522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
- added link hex_socket_head_cap_screw_m4x0_70_x_6__52230e09e6b8162f7a31d58ec48e066b_4, mass 0.00135184; collision mesh filename=package://assets/hex_socket_head_cap_screw_m4x0_70_x_6__522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; visual mesh filename=package://assets/hex_socket_head_cap_screw_m4x0_70_x_6__522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
- added link large_gear, mass 1e-09; collision mesh filename=package://assets/large_gear.stl; visual mesh filename=package://assets/large_gear.stl
- added link large_support, mass 1e-09; collision mesh filename=package://assets/large_support.stl; visual mesh filename=package://assets/large_support.stl
- added link small_gear_2, mass 1e-09; collision mesh filename=package://assets/small_gear.stl; visual mesh filename=package://assets/small_gear.stl
- added link socket_head_cap_screw__10_32_x_1__ce3b92dae7529e19d48acf72f7418474, mass 0.00513271; collision mesh filename=package://assets/socket_head_cap_screw__10_32_x_1__ce3b92da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; visual mesh filename=package://assets/socket_head_cap_screw__10_32_x_1__ce3b92da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
- added link socket_head_cap_screw__10_32_x_1__ce3b92dae7529e19d48acf72f7418474_2, mass 0.00513271; collision mesh filename=package://assets/socket_head_cap_screw__10_32_x_1__ce3b92da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; visual mesh filename=package://assets/socket_head_cap_screw__10_32_x_1__ce3b92da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
- added link socket_head_cap_screw__10_32_x_1__ce3b92dae7529e19d48acf72f7418474_3, mass 0.00513271; collision mesh filename=package://assets/socket_head_cap_screw__10_32_x_1__ce3b92da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; visual mesh filename=package://assets/socket_head_cap_screw__10_32_x_1__ce3b92da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
- added link socket_head_cap_screw__10_32_x_1__ce3b92dae7529e19d48acf72f7418474_4, mass 0.00513271; collision mesh filename=package://assets/socket_head_cap_screw__10_32_x_1__ce3b92da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; visual mesh filename=package://assets/socket_head_cap_screw__10_32_x_1__ce3b92da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
- added link spacer, mass 1e-09; collision mesh filename=package://assets/spacer.stl; visual mesh filename=package://assets/spacer.stl
- added link spacer_2, mass 1e-09; collision mesh filename=package://assets/spacer.stl; visual mesh filename=package://assets/spacer.stl
- added link spacer_3, mass 1e-09; collision mesh filename=package://assets/spacer.stl; visual mesh filename=package://assets/spacer.stl
- added link spacer_4, mass 1e-09; collision mesh filename=package://assets/spacer.stl; visual mesh filename=package://assets/spacer.stl
- added link stepper_motor, mass 1e-09; collision mesh filename=package://assets/28byj_48_002.stl; collision mesh filename=package://assets/28byj_48_003.stl
- added link stepper_motor_2, mass 1e-09; collision mesh filename=package://assets/28byj_48_002.stl; collision mesh filename=package://assets/28byj_48_003.stl
- added link top_enclosure, mass 1e-09; collision mesh filename=package://assets/top_enclosure.stl; visual mesh filename=package://assets/top_enclosure.stl
Joints:
- added joint carriage: type revolute, parent 375__round_id__875__od_radial_bearing__217_3239, child spacer, origin xyz=0 0 0 rpy=-3.14159 -0 0.129164, axis 0 0 1, limit lower=-3.141592653589793 upper=3.141592653589793 effort=10 velocity=10
- added joint f0: type fixed, parent large_support, child 375__round_id__875__od_radial_bearing__217_3239_5, origin xyz=0.05334 0 0.06985 rpy=-1.5708 0 1.5708, axis 0 0 1, limit effort=10 velocity=10
- added joint f1: type fixed, parent spacer, child 375__round_id__875__od_radial_bearing__217_3239_2, origin xyz=0 0 -0.00254 rpy=0 0 0, axis 0 0 1, limit effort=10 velocity=10
- added joint f3: type fixed, parent large_support, child stepper_motor, origin xyz=-0.06754 0.0175 0.06195 rpy=1.5708 -0 1.5708, axis 0 0 1, limit effort=10 velocity=10
- added joint f4: type fixed, parent large_support, child stepper_motor_2, origin xyz=0.06754 0.0175 0.06195 rpy=-1.5708 -0 1.5708, axis 0 0 1, limit effort=10 velocity=10
- added joint f5: type fixed, parent large_gear, child headtop, origin xyz=0 -0 0.0351276 rpy=3.14159 -0 -0, axis 0 0 1, limit effort=10 velocity=10
- added joint f6: type fixed, parent bottom_enclosure, child top_enclosure, origin xyz=0.00762 0.03175 0.09652 rpy=1.5708 -1.5708 0, axis 0 0 1, limit effort=10 velocity=10
- added joint f7: type fixed, parent bottom_enclosure, child spacer_4, origin xyz=-0 -0 0.0127 rpy=3.14159 0 0, axis 0 0 1, limit effort=10 velocity=10
- added joint f8: type fixed, parent stepper_motor_2, child hex_socket_head_cap_screw_m4x0_70_x_6__52230e09e6b8162f7a31d58ec48e066b_4, origin xyz=-0.035 -0 -0.0008 rpy=-3.14159 0 1.5708, axis 0 0 1, limit effort=10 velocity=10
- added joint f9: type fixed, parent top_enclosure, child socket_head_cap_screw__10_32_x_1__ce3b92dae7529e19d48acf72f7418474_4, origin xyz=-0 0.01524 -0.0127 rpy=3.14159 -0 -0, axis 0 0 1, limit effort=10 velocity=10
- added joint leftGear: type revolute, parent spacer_3, child small_gear, origin xyz=-0 -0 -0.00254 rpy=-0 -0 0.700636, axis 0 0 1, limit lower=-3.141592653589793 upper=3.141592653589793 effort=10 velocity=10
- added joint rightGear: type revolute, parent spacer_4, child small_gear_2, origin xyz=0 -0 -0.00254 rpy=-0 -0 1.78704, axis 0 0 1, limit lower=-3.141592653589793 upper=3.141592653589793 effort=10 velocity=10, mimic joint=topgear multiplier=-0.5555555555555556
- added joint topgear: type revolute, parent top_enclosure, child large_gear, origin xyz=-0.04572 0.00762 0.00508 rpy=3.14159 0 0.389242, axis 0 0 1, limit lower=-3.141592653589793 upper=3.141592653589793 effort=10 velocity=10, mimic joint=leftGear multiplier=-0.5555555555555556
